File: hardware/esp32-cc1101-multiband.kicad_pcb (KiCad board)
At the start: 4 copper layers, 90 x 36 mm, 107 parts, among them J1 USB-C USB2.0, J2 SMA FEMALE VERTICAL 50 OHM, J3 EXPANSION (DNP), Q1 MMBT3904, Q2 MMBT3904, SW1 RESET, SW2 BOOT, U1 ESP32-WROOM-32E-N8, U2 CC1101RGPR, U3 BGS13SN8E6327XTSA1, U4 BGS13SN8E6327XTSA1, U5 CP2102N-A02-GQFN24, U6 AP7361C-33E-13, Y1 ABM8-26.000MHZ-10-1-U-T

Commit message: Develop A3 routed prototype candidate with power and RF redesign
Parts:
- removed R40: 0R, R_0402_1005Metric
- added C13: 22uF 25V, C_1206_3216Metric, F.Cu at (23.0, 8.50)
- added C14: 100nF, C_0402_1005Metric, F.Cu at (16.1, 2.50)
- added C70: 10nF, C_0402_1005Metric, F.Cu at (12.6, 11.3)
- added C71: 100nF, C_0402_1005Metric, F.Cu at (27.7, 28.8)
- added J4: POWER ARM AUTO / EXT, PinHeader_1x03_P2.54mm_Vertical, F.Cu at (7.80, 1.90)
- added L1: 4.7uH XAL4030, L_Coilcraft_XAL4030-XXX, F.Cu at (19.2, 5.50)
- added R33: 10k pullup, R_0603_1608Metric, F.Cu at (56.5, 27.5)
- added R34: 10k pullup, R_0603_1608Metric, F.Cu at (74.0, 28.5)
- added R35: 10k pullup, R_0603_1608Metric, F.Cu at (77.0, 28.5)
- added R60: 49.9R 1%, R_0402_1005Metric, F.Cu at (64.0, 21.3)
- added R61: 49.9R 1%, R_0402_1005Metric, F.Cu at (78.3, 14.7)
- added R70: 10k, R_0603_1608Metric, F.Cu at (18.0, 12.3)
- added R71: 100k, R_0603_1608Metric, F.Cu at (18.0, 14.3)
- added U7: TPS22918DBVR, SOT-23-6, F.Cu at (9.50, 9.80)
- added U8: SN74LVC2G125DCTR, SSOP-8_2.95x2.8mm_P0.65mm, F.Cu at (24.3, 30.0)
- C1: value 10uF 10V -> 22uF 25V; footprint C_0805_2012Metric -> C_1206_3216Metric
- C2: value 22uF 6.3V -> 22uF 25V; footprint C_0805_2012Metric -> C_1206_3216Metric
- C8: value 4.7uF -> DNP
- D3: value STATUS BLUE -> STATUS GREEN
- F1: value 500mA PTC -> 750mA PTC
- R12: value 1k -> 330R 1%
- R13: value 2.2k -> 330R 1%
- R31, R32: value 100k pulldown -> 10k pullup
- U3, U4: value BGS13SN8E6327XTSA1 -> PE42442A-Z; footprint Infineon_PG-TSNP-8-1 -> pSemi_PE42442_QFN24
- U6: value AP7361C-33E-13 -> AP63203WU-7; footprint SOT-223-3_TabPin2 -> Diodes_TSOT26
- moved C54 16.1 mm to (86.5, 9.50)
- moved C53 15.9 mm to (84.0, 9.50)
- moved D5 14.2 mm to (88.2, 11.5), turned to 0 degrees
- moved C9 14.2 mm to (10.5, 13.0), turned to 0 degrees
- moved C52 12.1 mm to (81.5, 9.50)
- moved R41 8.49 mm to (85.0, 11.0)
- moved L52 8.43 mm to (83.0, 11.0)
- moved C2 7.93 mm to (18.7, 9.50)
- moved C61 4.56 mm to (78.2, 22.7), turned to -90 degrees
- moved C60 4.52 mm to (64.4, 14.8)
- moved C31 4.48 mm to (47.5, 22.9), turned to 180 degrees
- moved D2 4.21 mm to (6.80, 9.00), turned to 90 degrees
- moved C46 4.06 mm to (71.1, 11.0)
- moved C32 3.18 mm to (52.8, 24.5)
- moved U6 2.69 mm to (14.5, 5.50)
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Connections:
- C1 pad 1: /VBUS_PROTECTED -> /VBUS_SWITCHED
- C3 pad 1: /+3V3 -> /+3V3_USB
- C4 pad 1: /+3V3 -> /+3V3_USB
- C44 pad 1: /BALUN_M2 -> /RF_SWITCH_IN
- C6 pad 1: /+3V3 -> /+3V3_USB
- C7 pad 1: /+3V3 -> /VBUS_PROTECTED
- C8 pad 1: /+3V3 -> /+3V3_USB
- C9 pad 1: /+3V3 -> /VBUS_PROTECTED
- J3 pad 6: /EXP_GPIO16 -> /RF_OUT0
- J3 pad 7: /EXP_GPIO17 -> /RF_OUT1
- L41 pad 2: /BALUN_M2 -> /RF_SWITCH_IN
- R3 pad 2: /+3V3 -> /+3V3_USB
- R31 pad 2: /GND -> /+3V3_RF
- R32 pad 2: /GND -> /+3V3_RF
- U1 pad 26: unconnected-(U1-IO4-Pad26) -> /RF_DISABLE
- U1 pad 27: /EXP_GPIO16 -> /RF_OUT0
- U1 pad 28: /EXP_GPIO17 -> /RF_OUT1
- U3 pad 1: /+3V3_RF -> /GND
- U3 pad 2: /RF_SW0 -> /GND
- U3 pad 3: /RF_SW1 -> /GND
- U3 pad 4: /RF_868_915_IN -> /GND
- U3 pad 5: /RF_315_IN -> /U3_RF4_TERM
- U3 pad 6: /RF_SWITCH_IN -> /GND
- U3 pad 7: /RF_433_IN -> /GND
- U3 pad 8: /GND -> /RF_868_915_IN
- U4 pad 1: /+3V3_RF -> /GND
- U4 pad 2: /RF_SW0 -> /GND
- U4 pad 3: /RF_SW1 -> /GND
- U4 pad 4: /RF868_B -> /GND
- U4 pad 5: /RF_315_OUT -> /U4_RF4_TERM
- U4 pad 6: /RF_COMBINED -> /GND
- U4 pad 7: /RF_433_OUT -> /GND
- U4 pad 8: /GND -> /RF_315_OUT
- U5 pad 15: unconnected-(U5-~{SUSPEND}-Pad15) -> /USB_ACTIVE
- U5 pad 20: /UART_TX_ESP -> /UART_RX_USB
- U5 pad 21: /UART_RX_ESP -> /UART_TX_USB
- U5 pad 5: /+3V3 -> /+3V3_USB
- U5 pad 6: /+3V3 -> /+3V3_USB
- U5 pad 7: /+3V3 -> /VBUS_PROTECTED
- U6 pad 1: /VBUS_PROTECTED -> /+3V3
- U6 pad 2: /GND -> /VBUS_SWITCHED
- U6 pad 3: /+3V3 -> /VBUS_SWITCHED
Other:
- board text added: "CONFIGURE USB BEFORE FITTING J4"
- board text added: "ESP32 + CC1101 MULTIBAND REV A3"
- board text added: "J4: 1-2 AUTO / 2-3 EXT"
- board text removed: "ESP32 + CC1101 MULTIBAND REV A2"
