File: hardware/esp32-cc1101-multiband.kicad_sch (KiCad schematic)
At the start: 103 parts, among them J1 USB-C USB2.0, J2 SMA FEMALE VERTICAL 50 OHM, J3 EXPANSION (DNP), Q1 MMBT3904, Q2 MMBT3904, SW1 RESET, SW2 BOOT, U1 ESP32-WROOM-32E-N8, U2 CC1101RGPR, U3 BGS13SN8E6327XTSA1, U4 BGS13SN8E6327XTSA1, U5 CP2102N-A02-GQFN24, U6 AP7361C-33E-13, Y1 ABM8-26.000MHZ-10-1-U-T

Commit message: Develop A3 routed prototype candidate with power and RF redesign
Parts:
- removed R40: 0R, Resistor_SMD:R_0402_1005Metric, symbol Device:R
- removed U3, U4: BGS13SN8E6327XTSA1, ESP32_CC1101_RF:Infineon_PG-TSNP-8-1, symbol ESP32_CC1101:BGS13SN8
- removed U6: AP7361C-33E-13, Package_TO_SOT_SMD:SOT-223-3_TabPin2, symbol Regulator_Linear:AP7361C-33E
- added C13: 22uF 25V, Capacitor_SMD:C_1206_3216Metric, symbol Device:C
- added C14, C71: 100nF, Capacitor_SMD:C_0402_1005Metric, symbol Device:C
- added C70: 10nF, Capacitor_SMD:C_0402_1005Metric, symbol Device:C
- added J4: POWER ARM AUTO / EXT, Connector_PinHeader_2.54mm:PinHeader_1x03_P2.54mm_Vertical, symbol Connector_Generic:Conn_01x03
- added L1: 4.7uH XAL4030, Inductor_SMD:L_Coilcraft_XAL4030-XXX, symbol Device:L
- added R33, R34, R35: 10k pullup, Resistor_SMD:R_0603_1608Metric, symbol Device:R
- added R60, R61: 49.9R 1%, Resistor_SMD:R_0402_1005Metric, symbol Device:R
- added R70: 10k, Resistor_SMD:R_0603_1608Metric, symbol Device:R
- added R71: 100k, Resistor_SMD:R_0603_1608Metric, symbol Device:R
- added U3, U4: PE42442A-Z, ESP32_CC1101_RF:pSemi_PE42442_QFN24, symbol ESP32_CC1101:PE42442
- added U6: AP63203WU-7, ESP32_CC1101_RF:Diodes_TSOT26, symbol ESP32_CC1101:AP63203
- added U7: TPS22918DBVR, Package_TO_SOT_SMD:SOT-23-6, symbol ESP32_CC1101:TPS22918
- added U8: SN74LVC2G125DCTR, Package_SO:SSOP-8_2.95x2.8mm_P0.65mm, symbol ESP32_CC1101:SN74LVC2G125
- C1: value 10uF 10V -> 22uF 25V; footprint Capacitor_SMD:C_0805_2012Metric -> Capacitor_SMD:C_1206_3216Metric
- C2: value 22uF 6.3V -> 22uF 25V; footprint Capacitor_SMD:C_0805_2012Metric -> Capacitor_SMD:C_1206_3216Metric
- C8: value 4.7uF -> DNP
- D3: value STATUS BLUE -> STATUS GREEN
- F1: value 500mA PTC -> 750mA PTC
- R12: value 1k -> 330R 1%
- R13: value 2.2k -> 330R 1%
- R31, R32: value 100k pulldown -> 10k pullup
Connections:
- net BALUN_M2 is gone; now on net RF_SWITCH_IN: C44.1, L41.2
- net +3V3: now also C13.1, C71.1, L1.2, U6.1 (FB), U8.8 (VCC); no longer C3.1, C4.1, C6.1, C7.1, C8.1, C9.1, R3.2, U5.5 (VIO), U5.6 (VDD), U5.7 (VREGIN)
- net +3V3_RF: now also R31.2, R32.2, R33.2, R34.2, R35.2, U3.16 (VDD), U4.16 (VDD)
- net GND: now also C13.2, C70.2, C71.2, R60.2, R61.2, R70.2, R71.2, U3.1 (GND), U3.10 (GND), U3.12 (GND), U3.13 (GND), U3.15 (GND), U3.2 (GND), U3.20 (VSS_EXT), U3.21 (GND), U3.23 (GND), U3.24 (GND), U3.25 (EP_GND), U3.3 (GND), U3.4 (GND), U3.6 (GND), U3.7 (GND), U3.9 (GND), U4.1 (GND), U4.10 (GND), U4.12 (GND), U4.13 (GND), U4.15 (GND), U4.2 (GND), U4.20 (VSS_EXT), U4.21 (GND), U4.23 (GND), U4.24 (GND), U4.25 (EP_GND), U4.3 (GND), U4.4 (GND), U4.6 (GND), U4.7 (GND), U4.9 (GND), U6.4 (GND), U7.2 (GND), U8.1 (~{1OE}), U8.4 (GND), U8.7 (~{2OE}); no longer R31.2, R32.2
- net RF868_B: now also U4.14 (RF1)
- net RF_315_IN: now also U3.14 (RF1)
- net RF_315_OUT: now also U4.8 (RF3)
- net RF_433_IN: now also U3.11 (RF2)
- net RF_433_OUT: now also U4.11 (RF2)
- net RF_868_915_IN: now also U3.8 (RF3)
- net RF_COMBINED: now also U4.22 (RFC)
- net RF_SW0: now also U3.17 (V1)
- net RF_SW1: now also U3.18 (V2)
- net RF_SWITCH_IN: now also U3.22 (RFC)
- net UART_RX_ESP: now also U8.6 (1Y); no longer U5.21 (TXD)
- net UART_TX_ESP: now also U8.5 (2A); no longer U5.20 (RXD)
- net VBUS_PROTECTED: now also C7.1, C9.1, U5.7 (VREGIN), U7.1 (VIN); no longer C1.1
- net USB_ACTIVE: now reaches U5.15 (~{SUSPEND})
- net USB_ACTIVE: now also J4.1 (Pin_1), R70.1
- net RF_DISABLE: now reaches U1.26 (IO4)
- net RF_DISABLE: now also R33.1, U3.19 (V3), U4.19 (V3)
- net EXP_GPIO16 renamed RF_OUT0
- net RF_OUT0: now also R34.1, U4.17 (V1)
- net EXP_GPIO17 renamed RF_OUT1
- net RF_OUT1: now also R35.1, U4.18 (V2)
- new net +3V3_USB: C3.1, C4.1, C6.1, C8.1, J4.3 (Pin_3), R3.2, U5.5 (VIO), U5.6 (VDD)
- new net BUCK_BST: C14.1, U6.6 (BST)
- new net BUCK_SW: C14.2, L1.1, U6.5 (SW)
- new net MAIN_POWER_EN: J4.2 (Pin_2), R71.1, U7.3 (ON)
- new net POWER_SLEW: C70.1, U7.4 (CT)
- new net U3_RF4_TERM: R60.1, U3.5 (RF4)
- new net U4_RF4_TERM: R61.1, U4.5 (RF4)
- new net UART_RX_USB: U5.20 (RXD), U8.3 (2Y)
- new net UART_TX_USB: U5.21 (TXD), U8.2 (1A)
- new net VBUS_SWITCHED: C1.1, U6.2 (EN), U6.3 (VIN), U7.5 (QOD), U7.6 (VOUT)
- no-connect marks 23 -> 21
Other:
- note added: "J4: ship UNJUMPERED. Configure CP2102N for 500mA before AUTO (1-2). EXT (2-3) only with a known adequate 5V source; no USB power negotiation."
